File: pcb/chaski.kicad_pcb (KiCad board)
At the start: 2 copper layers, 271.7 x 145.2 mm, 103 parts

Commit message: fix: NFC1 and NFC2 were mis-labeled on the PCB
Connections:
- PAD3 pad 1: NFC2 -> NFC1
- PAD4 pad 1: NFC1 -> NFC2
- SW11 pad 1: NFC1 -> NFC2
- SW12 pad 1: NFC2 -> NFC1
- SW17 pad 1: NFC1 -> NFC2
- SW18 pad 1: NFC2 -> NFC1
- SW23 pad 1: NFC1 -> NFC2
- SW24 pad 1: NFC2 -> NFC1
- SW29 pad 1: NFC1 -> NFC2
- SW30 pad 1: NFC2 -> NFC1
- SW35 pad 1: NFC1 -> NFC2
- SW36 pad 1: NFC2 -> NFC1
- SW41 pad 1: NFC1 -> NFC2
- SW42 pad 1: NFC2 -> NFC1
- SW5 pad 1: NFC1 -> NFC2
- SW6 pad 1: NFC2 -> NFC1
Routing:
- net NFC2: track 328.1 -> 328.3 mm, vias 1 -> 2
- net NFC1: track 328.3 -> 328.1 mm, vias 2 -> 1
