File: pcb/gigas.kicad_pcb (KiCad board)
At the start: 2 copper layers, 228.8 x 117.8 mm, 92 parts

Commit message: fix: NFC1 and NFC2 were mis-labeled on the PCB
Connections:
- PAD3 pad 1: NFC2 -> NFC1
- PAD4 pad 1: NFC1 -> NFC2
- S29 pad 1: NFC1 -> NFC2
- S31 pad 1: NFC1 -> NFC2
- SKRH1 pad COMMON: NFC2 -> NFC1
Routing:
- net NFC2: track 59.1 -> 112.8 mm, vias 0 -> 1
- net NFC1: track 112.8 -> 59.1 mm, vias 1 -> 0
Other:
- board text added: "NFC1-P4"
- board text added: "NFC1-P6"
- board text added: "NFC1-P7"
- board text removed: "NFC2-P4"
- board text removed: "NFC2-P6"
- board text removed: "NFC2-P7"
Changed lines of the file:
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@@
 			(outputformat 1)
 			(mirror no)
-			(drillshape 1)
+			(drillshape 0)
 			(scaleselection 1)
-			(outputdirectory "")
+			(outputdirectory "gigas")
 		)
 	)
@@
 		)
 		(duplicate_pad_numbers_are_jumpers no)
-		(fp_text user "NFC1"
+		(fp_text user "NFC2"
 			(at 0 2 0)
 			(layer "B.SilkS")
@@
 			(layers "*.Cu" "*.Mask")
 			(remove_unused_layers no)
-			(net "NFC1")
+			(net "NFC2")
 		)
 		(pad "1" thru_hole circle
@@
 			(layers "*.Cu" "F.Mask")
 			(remove_unused_layers no)
-			(net "NFC1")
+			(net "NFC2")
 		)
 		(pad "1" thru_hole circle
@@
 			(layers "*.Cu" "B.Mask")
 			(remove_unused_layers no)
-			(net "NFC1")
+			(net "NFC2")
 		)
 		(embedded_fonts no)
@@
 		)
 		(duplicate_pad_numbers_are_jumpers no)
-		(fp_text user "NFC2"
+		(fp_text user "NFC1"
 			(at 0 2 0)
 			(layer "B.SilkS")
@@
 			(layers "*.Cu" "*.Mask")
 			(remove_unused_layers no)
-			(net "NFC2")
+			(net "NFC1")
 		)
 		(pad "1" thru_hole circle
@@
 			(layers "*.Cu" "F.Mask")
 			(remove_unused_layers no)
-			(net "NFC2")
+			(net "NFC1")
 		)
 		(pad "1" thru_hole circle
@@
 			(layers "*.Cu" "B.Mask")
 			(remove_unused_layers no)
-			(net "NFC2")
+			(net "NFC1")
 		)
 		(embedded_fonts no)
@@
 			(size 1.35 1)
 			(layers "F.Cu" "F.Mask" "F.Paste")
-			(net "NFC2")
+			(net "NFC1")
 		)
 		(pad "D" smd rect
@@
 			(size 2.6 2.6)
 			(layers "B.Cu" "B.Mask" "B.Paste")
-			(net "NFC1")
+			(net "NFC2")
 		)
 		(pad "2" smd rect
@@
 			(size 2.6 2.6)
 			(layers "B.Cu" "B.Mask" "B.Paste")
-			(net "NFC1")
+			(net "NFC2")
 		)
 		(pad "2" smd rect
@@
 		)
 	)
-	(gr_text "NFC1-P5"
+	(gr_text "NFC2-P5"
 		(at 116.96087 118.116353 -37.5)
 		(layer "B.SilkS")
@@
 		)
 	)
-	(gr_text "NFC2-P6"
+	(gr_text "NFC1-P6"
 		(at 142.37026 117.715046 0)
 		(layer "B.SilkS")
@@
 		)
 	)
-	(gr_text "NFC2-P8"
+	(gr_text "NFC1-P8"
 		(at 144.74526 112.965046 0)
 		(layer "B.SilkS")
@@
 		)
 	)
-	(gr_text "NFC2-P4"
+	(gr_text "NFC1-P4"
 		(at 151.87026 108.215046 0)
 		(layer "B.SilkS")
@@
 		)
 	)
-	(gr_text "NFC2-P7"
+	(gr_text "NFC1-P7"
 		(at 151.87026 127.215046 0)
 		(layer "B.SilkS")
@@
 		)
 	)
-	(gr_text "NFC2-P5"
+	(gr_text "NFC1-P5"
 		(at 161.37026 117.715046 0)
 		(layer "B.SilkS")
@@
 		)
 	)
-	(gr_text "NFC1-P8"
+	(gr_text "NFC2-P8"
 		(at 177.735422 125.056234 37.5)
 		(layer "B.SilkS")
@@
 		(width 0.2)
 		(layer "F.Cu")
-		(net "NFC1")
+		(net "NFC2")
 	)
 	(segment
@@
 		(width 0.2)
 		(layer "F.Cu")
-		(net "NFC1")
+		(net "NFC2")
 	)
 	(via
@@
 		(drill 0.3)
 		(layers "F.Cu" "B.Cu")
-		(net "NFC1")
+		(net "NFC2")
 	)
 	(segment
@@
 		(width 0.2)
 		(layer "B.Cu")
-		(net "NFC1")
+		(net "NFC2")
 	)
 	(segment
@@
 		(width 0.2)
 		(layer "B.Cu")
-		(net "NFC1")
+		(net "NFC2")
 	)
 	(segment
@@
 		(width 0.2)
 		(layer "B.Cu")
-		(net "NFC1")
+		(net "NFC2")
 	)
 	(segment
@@
 		(width 0.2)
 		(layer "B.Cu")
-		(net "NFC1")
+		(net "NFC2")
 	)
 	(segment
@@
 		(width 0.2)
 		(layer "B.Cu")
-		(net "NFC1")
+		(net "NFC2")
 	)
 	(segment
@@
 		(width 0.2)
 		(layer "B.Cu")
-		(net "NFC1")
+		(net "NFC2")
 	)
 	(segment
@@
 		(width 0.2)
 		(layer "B.Cu")
-		(net "NFC1")
+		(net "NFC2")
 	)
 	(segment
@@
 		(width 0.2)
 		(layer "F.Cu")
-		(net "NFC2")
+		(net "NFC1")
 	)
 	(segment
@@
 		(width 0.2)
 		(layer "F.Cu")
-		(net "NFC2")
+		(net "NFC1")
 	)
 	(segment
@@
 		(width 0.2)
 		(layer "F.Cu")
-		(net "NFC2")
+		(net "NFC1")
 	)
 	(segment
@@
 		(width 0.2)
 		(layer "F.Cu")
-		(net "NFC2")
+		(net "NFC1")
 	)
 	(segment
@@
 		(width 0.2)
 		(layer "F.Cu")
-		(net "NFC2")
+		(net "NFC1")
 	)
 	(segment
@@
 		(width 0.2)
 		(layer "F.Cu")
-		(net "NFC2")
+		(net "NFC1")
 	)
 	(segment
